File: electronics/caiman.kicad_pcb (KiCad board)
At the start: 2 copper layers, 90.9 x 93.9 mm, 132 parts, among them J1 Conn_01x03_Pin, J10 Conn_01x04_Pin, J11 Conn_01x04_Pin, J12 Conn_01x04_Pin, J13 Micro_SD_Card, J14 50 ohm, J15 Conn_01x03_Pin, J2 Conn_01x04_Pin, J3 Conn_01x04_Pin, J4 Conn_01x03_Pin, J5 Conn_01x04_Pin, J6 Conn_01x04_Pin, J7 Conn_01x02_Pin, J8 Conn_01x02_Pin, J9 Conn_01x02_Pin, Q1 Q_PMOS-E_Generic_SSSGD, Q2 AON6262E, U1 AP63205WU, U10 SN74LV1T34DBV, U2 AP63203WU, U3 US1881, U4 LM74700, U5 LPS22HBTR, U6 LIS2MDLTR, U7 STM32F765VITx, U8 LSM6DSO, U9 nRF24L01P, Y1 25MHz, Y2 16MHz

Commit message: Updating the PCB
Parts:
- added JP1: SolderJumper_2_Open, Jumper:SolderJumper-2_P1.3mm_Open_TrianglePad1.0x1.5mm, B.Cu at (146.6, 63.5)
- added R12: 10k, Resistor_SMD:R_0402_1005Metric, B.Cu at (145.4, 64.8)
- C10, C9: value 0.1uF -> 0.1uF, 50V; footprint Capacitor_SMD:C_0603_1608Metric -> Capacitor_SMD:C_0805_2012Metric
- C11: value 47uF -> 47uF, 50v
- C3: value 10uF -> 10uF, 50v; footprint Capacitor_SMD:C_0603_1608Metric -> Capacitor_SMD:C_0805_2012Metric
- C4, C5, C7, C8: value 22uF -> 22uF, 16V
- C6: value 10uF -> 10uF, 16v; footprint Capacitor_SMD:C_0603_1608Metric -> Capacitor_SMD:C_0805_2012Metric
- L1: value 3.3uH -> 4.7uH
- L2: value 2.2uH -> 3.9uH
- R7: value 27k -> 10k
- Y1: value 25MHz -> 8MHz
- moved C16 2.88 mm to (149.6, 63.3), turned to 45 degrees
- renumbered R12 to R13, R13 to R14, R14 to R15, R15 to R16, R16 to R17, R17 to R18, R18 to R19, R19 to R20, R20 to R21, R21 to R22, R22 to R23, R23 to R24, R24 to R25, R25 to R26, R26 to R27, R27 to R28, R28 to R29, R29 to R30, R30 to R31, R31 to R32
Connections:
- R1 pad 1: Net-(U1-EN) -> VCC
- R1 pad 2: VCC -> Net-(U1-EN)
- R2 pad 1: VCC -> Net-(U1-EN)
- U7 pad 94: unconnected-(U7-BOOT0-Pad94) -> Net-(JP1-B)
Routing:
- net VCC: track 24.8 -> 36.0 mm
- net +3V3: track 300.6 -> 305.7 mm
- net Net-(JP1-B): track 0.00 -> 4.56 mm
- net /NRST: track 35.4 -> 36.9 mm
- net Net-(U1-EN): track 3.88 -> 4.91 mm
- net Net-(U9-XC1): track 5.15 -> 5.81 mm
- net Net-(U9-XC2): track 5.18 -> 5.84 mm
- net Net-(C16-Pad1): track 2.44 -> 1.85 mm
- net GND: vias 151 -> 157
