File: electronics/_restore_backup_2026-06-08T14-48-05-926/caiman.kicad_pcb (KiCad board)
At the start: 2 copper layers, 90.9 x 93.9 mm, 134 parts, among them J1 Conn_01x03_Pin, J10 Conn_01x04_Pin, J11 Conn_01x04_Pin, J12 Conn_01x04_Pin, J13 Micro_SD_Card, J14 50 ohm, J15 Conn_01x03_Pin, J2 Conn_01x04_Pin, J3 Conn_01x04_Pin, J4 Conn_01x03_Pin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

Commit message: DRC Clean
Routing:
- net /I2C2_SDA: track 95.5 -> 94.3 mm
- net /VCHG: track 93.1 -> 92.1 mm
- net GND: track 22.3 -> 21.5 mm
